File: Larson15cm_1.sch (KiCad schematic (older format))
At the start: 19 parts

Commit message: C code added. Slightly broken at the moment. WIP
Parts:
- gave numbers to parts that had none: 3
Changed lines of the file:
@@
-EESchema Schematic File Version 2  date 26/08/2013 20:45:56
+EESchema Schematic File Version 2  date 26/08/2013 21:21:07
 LIBS:power
 LIBS:device
@@
 	6225 2050 6225 2325
 $Comp
-L GND #PWR?
+L GND #PWR3
 U 1 1 521BAF71
 P 6000 2700
-F 0 "#PWR?" H 6000 2700 30  0001 C CNN
+F 0 "#PWR3" H 6000 2700 30  0001 C CNN
 F 1 "GND" H 6000 2630 30  0001 C CNN
 	1    6000 2700
@@
 $EndComp
 $Comp
-L SW_PUSH SW?
+L SW_PUSH SW1
 U 1 1 521BAF63
 P 5700 2700
-F 0 "SW?" H 5850 2810 50  0000 C CNN
+F 0 "SW1" H 5850 2810 50  0000 C CNN
 F 1 "SW_PUSH" H 5700 2620 50  0000 C CNN
 	1    5700 2700
@@
 $EndComp
 $Comp
-L GND #PWR?
+L GND #PWR4
 U 1 1 521BAC4F
 P 6225 2325
-F 0 "#PWR?" H 6225 2325 30  0001 C CNN
+F 0 "#PWR4" H 6225 2325 30  0001 C CNN
 F 1 "GND" H 6225 2255 30  0001 C CNN
 	1    6225 2325
@@
 PB2-5 are PWM Pins
 $Comp
-L AVR-ISP-6 CON?
+L AVR-ISP-6 CON1
 U 1 1 521BAA0B
 P 5550 1950
-F 0 "CON?" H 5470 2190 50  0000 C CNN
+F 0 "CON1" H 5470 2190 50  0000 C CNN
 F 1 "AVR-ISP-6" H 5310 1720 50  0000 L BNN
 F 2 "AVR-ISP-6" V 5030 1990 50  0001 C CNN
@@
 $EndComp
 $Comp
-L ATTINY2313-P IC?
+L ATTINY2313-P IC1
 U 1 1 521BA8AA
 P 3150 2150
-F 0 "IC?" H 2300 3100 60  0000 C CNN
+F 0 "IC1" H 2300 3100 60  0000 C CNN
 F 1 "ATTINY2313-P" H 3750 1300 60  0000 C CNN
 F 2 "DIP20" H 2350 1300 60  0001 C CNN
@@
 $EndComp
 $Comp
-L GND #PWR01
+L GND #PWR2
 U 1 1 4F684FA2
 P 3150 3150
-F 0 "#PWR01" H 3150 3150 30  0001 C CNN
+F 0 "#PWR2" H 3150 3150 30  0001 C CNN
 F 1 "GND" H 3150 3080 30  0001 C CNN
 	1    3150 3150
@@
 $EndComp
 $Comp
-L +3.3V #PWR02
+L +3.3V #PWR1
 U 1 1 4F684F91
 P 3150 1050
-F 0 "#PWR02" H 3150 1010 30  0001 C CNN
+F 0 "#PWR1" H 3150 1010 30  0001 C CNN
 F 1 "+3.3V" H 3150 1160 30  0000 C CNN
 	1    3150 1050
