File: Larson.sch (KiCad schematic (older format))
At the start: 17 parts, among them IC1 ATTINY85-P

Commit message: House Keeping
Parts:
- removed IC1: ATTINY85-P, DIP8, symbol ATTINY85-P
- added CON1: AVR-ISP-6, AVR-ISP-6, symbol AVR-ISP-6
- added IC1: ATTINY2313-P, DIP20, symbol ATTINY2313-P
- added SW1: SW_PUSH, symbol SW_PUSH
Connections:
- wire segments 43 -> 79
Other:
- note added: "PB2-5 are PWM Pins"
Changed lines of the file:
@@
-EESchema Schematic File Version 2  date 14/05/2012 20:33:47
+EESchema Schematic File Version 2  date 09/09/2013 14:06:59
 LIBS:power
 LIBS:device
@@
 LIBS:contrib
 LIBS:valves
+LIBS:Larson15cm_1-cache
 EELAYER 25  0
 EELAYER END
@@
 Sheet 1 1
 Title "noname.sch"
-Date "3 apr 2012"
+Date "9 sep 2013"
 Rev ""
 Comp ""
@@
 $EndDescr
 Wire Wire Line
-	1300 3600 6950 3600
-Wire Wire Line
-	1400 3700 6200 3700
-Wire Wire Line
-	1500 3800 5450 3800
-Wire Wire Line
-	3700 4800 7200 4800
-Wire Wire Line
-	2700 4700 1500 4700
-Wire Wire Line
-	2700 4600 6700 4600
-Wire Wire Line
-	2200 4500 6450 4500
+	4300 2750 4350 2750
+Wire Wire Line
+	4350 2750 4350 3250
+Wire Wire Line
+	4350 3250 2050 3250
+Wire Wire Line
+	6225 2325 6225 2050
+Wire Wire Line
+	6225 2050 5675 2050
+Wire Wire Line
+	4300 1850 4850 1850
+Wire Wire Line
+	4850 1850 4850 1625
+Wire Wire Line
+	4850 1625 5950 1625
+Wire Wire Line
+	5950 1625 5950 1950
+Wire Wire Line
+	5950 1950 5675 1950
+Wire Wire Line
+	5425 1950 5325 1950
+Wire Wire Line
+	5325 1950 5325 2050
+Wire Wire Line
+	5325 2050 4300 2050
+Wire Wire Line
+	2050 2700 1300 2700
+Wire Wire Line
+	2050 2700 2050 3250
+Wire Wire Line
+	1900 2900 1500 2900
+Wire Wire Line
+	1900 2900 1900 3400
+Wire Wire Line
+	1900 3400 4550 3400
+Wire Wire Line
+	4550 3400 4550 1650
+Wire Wire Line
+	4550 1650 4300 1650
+Wire Wire Line
+	1800 3500 4650 3500
+Wire Wire Line
+	1800 3500 1800 3000
+Wire Wire Line
+	3200 4800 1600 4800
+Wire Wire Line
+	3200 4700 6950 4700
+Wire Wire Line
+	2200 4600 1400 4600
+Wire Wire Line
+	1700 4500 1300 4500
+Connection ~ 1400 3700
+Connection ~ 1600 3900
+Wire Wire Line
+	1600 3900 4700 3900
+Wire Wire Line
+	1600 4800 1600 3000
+Wire Wire Line
+	1400 4600 1400 2800
+Connection ~ 5200 4800
+Connection ~ 5450 4500
+Wire Wire Line
+	1300 4500 1300 2700
+Connection ~ 6950 4000
+Wire Wire Line
+	6950 4000 6950 3600
+Connection ~ 5450 4000
+Wire Wire Line
+	5450 4000 5450 3800
+Wire Wire Line
+	5450 4500 5450 4400
+Wire Wire Line
+	6700 4400 6700 4600
+Wire Wire Line
+	4700 4600 4700 4400
+Wire Wire Line
+	5950 4700 5950 4400
+Wire Wire Line
+	7200 4400 7200 4800
+Wire Wire Line
+	5200 4800 5200 4400
+Wire Wire Line
+	6700 4000 7200 4000
+Wire Wire Line
+	5200 4000 5700 4000
+Wire Wire Line
+	4450 4000 4950 4000
+Wire Wire Line
+	5950 4000 6450 4000
+Connection ~ 4700 4000
+Wire Wire Line
+	4700 3900 4700 4000
+Wire Wire Line
+	6200 4800 6200 4400
+Wire Wire Line
+	4950 4700 4950 4400
+Wire Wire Line
+	6950 4700 6950 4400
+Wire Wire Line
+	5700 4600 5700 4400
+Wire Wire Line
+	4450 4500 4450 4400
+Wire Wire Line
+	6450 4400 6450 4500
+Wire Wire Line
+	6200 4000 6200 3700
+Connection ~ 6200 4000
+Wire Wire Line
+	1600 3000 1800 3000
+Connection ~ 4450 4500
+Connection ~ 5700 4600
+Connection ~ 5950 4700
+Connection ~ 6200 4800
+Connection ~ 4700 4600
+Connection ~ 4950 4700
+Wire Wire Line
+	1500 2900 1500 4700
+Connection ~ 1500 3800
 Connection ~ 1300 3600
-Connection ~ 1500 3800
-Wire Wire Line
-	1500 4700 1500 2900
-Connection ~ 4950 4700
-Connection ~ 4700 4600
-Connection ~ 6200 4800
-Connection ~ 5950 4700
-Connection ~ 5700 4600
-Connection ~ 4450 4500
-Wire Wire Line
-	4500 2700 4650 2700
-Wire Wire Line
-	1800 2800 1400 2800
-Wire Wire Line
-	1800 3000 1600 3000
-Connection ~ 6200 4000
-Wire Wire Line
-	6200 3700 6200 4000
-Wire Wire Line
-	6450 4500 6450 4400
-Wire Wire Line
-	4450 4500 4450 4400
-Wire Wire Line
-	5700 4600 5700 4400
-Wire Wire Line
-	6950 4400 6950 4700
-Wire Wire Line
-	4950 4700 4950 4400
-Wire Wire Line
-	6200 4800 6200 4400
-Wire Wire Line
-	4700 4000 4700 3900
-Connection ~ 4700 4000
-Wire Wire Line
-	5950 4000 6450 4000
-Wire Wire Line
-	4450 4000 4950 4000
-Wire Wire Line
-	5200 4000 5700 4000
-Wire Wire Line
-	6700 4000 7200 4000
-Wire Wire Line
-	5200 4800 5200 4400
-Wire Wire Line
-	7200 4800 7200 4400
-Wire Wire Line
-	5950 4700 5950 4400
-Wire Wire Line
-	4700 4600 4700 4400
-Wire Wire Line
-	6700 4600 6700 4400
-Wire Wire Line
-	5450 4500 5450 4400
-Wire Wire Line
-	5450 3800 5450 4000
-Connection ~ 5450 4000
-Wire Wire Line
-	6950 3600 6950 4000
-Connection ~ 6950 4000
-Wire Wire Line
-	1500 2900 1800 2900
-Wire Wire Line
-	1800 2700 1300 2700
-Wire Wire Line
-	1300 2700 1300 4500
-Wire Wire Line
-	4500 3200 4650 3200
-Wire Wire Line
-	4650 3200 4650 3250
-Connection ~ 5450 4500
-Connection ~ 5200 4800
-Wire Wire Line
-	1400 2800 1400 4600
-Wire Wire Line
-	1600 3000 1600 4800
-Wire Wire Line
-	4700 3900 1600 3900
-Connection ~ 1600 3900
-Connection ~ 1400 3700
-Wire Wire Line
-	1300 4500 1700 4500
-Wire Wire Line
-	1400 4600 2200 4600
-Wire Wire Line
-	6950 4700 3200 4700
-Wire Wire Line
-	1600 4800 3200 4800
+Wire Wire Line
+	6450 4500 2200 4500
+Wire Wire Line
+	6700 4600 2700 4600
+Wire Wire Line
+	1500 4700 2700 4700
+Wire Wire Line
+	7200 4800 3700 4800
+Wire Wire Line
+	5450 3800 1500 3800
+Wire Wire Line
+	6200 3700 1400 3700
+Wire Wire Line
+	6950 3600 1300 3600
+Wire Wire Line
+	4650 3500 4650 1550
+Wire Wire Line
+	4650 1550 4300 1550
+Wire Wire Line
+	4300 1750 4450 1750
+Wire Wire Line
+	4450 1750 4450 3300
+Wire Wire Line
+	4450 3300 2000 3300
+Wire Wire Line
+	2000 3300 2000 2800
+Wire Wire Line
+	2000 2800 1400 2800
+Wire Wire Line
+	4300 1950 5200 1950
+Wire Wire Line
+	5200 1950 5200 1850
+Wire Wire Line
+	5200 1850 5425 1850
+Wire Wire Line
+	5675 1850 5675 1000
+Wire Wire Line
+	5675 1000 3150 1000
+Wire Wire Line
+	5425 2050 5425 2225
+Wire Wire Line
+	5425 2225 4700 2225
+Wire Wire Line
+	4700 2225 4700 1075
+Wire Wire Line
+	4700 1075 2000 1075
+Wire Wire Line
+	2000 1075 2000 1350
+Wire Wire Line
+	4300 2450 5200 2450
+Wire Wire Line
+	5200 2450 5200 2700
+Wire Wire Line
+	5200 2700 5400 2700
 $Comp
 L GND #PWR01
+U 1 1 521BAF71
+P 6000 2700
+F 0 "#PWR01" H 6000 2700 30  0001 C CNN
+F 1 "GND" H 6000 2630 30  0001 C CNN
+	1    6000 2700
+	1    0    0    -1
+$EndComp
+$Comp
+L SW_PUSH SW1
+U 1 1 521BAF63
+P 5700 2700
+F 0 "SW1" H 5850 2810 50  0000 C CNN
+F 1 "SW_PUSH" H 5700 2620 50  0000 C CNN
+	1    5700 2700
+	1    0    0    -1
+$EndComp
+$Comp
+L GND #PWR02
+U 1 1 521BAC4F
+P 6225 2325
+F 0 "#PWR02" H 6225 2325 30  0001 C CNN
+F 1 "GND" H 6225 2255 30  0001 C CNN
+	1    6225 2325
+	1    0    0    -1
+$EndComp
+Text Notes 3075 2200 0    60   ~ 0
+PB2-5 are PWM Pins
+$Comp
+L AVR-ISP-6 CON1
+U 1 1 521BAA0B
+P 5550 1950
+F 0 "CON1" H 5470 2190 50  0000 C CNN
+F 1 "AVR-ISP-6" H 5310 1720 50  0000 L BNN
+F 2 "AVR-ISP-6" V 5030 1990 50  0001 C CNN
+	1    5550 1950
+	1    0    0    -1
+$EndComp
+$Comp
+L ATTINY2313-P IC1
+U 1 1 521BA8AA
+P 3150 2150
+F 0 "IC1" H 2300 3100 60  0000 C CNN
+F 1 "ATTINY2313-P" H 3750 1300 60  0000 C CNN
+F 2 "DIP20" H 2350 1300 60  0001 C CNN
+	1    3150 2150
+	1    0    0    -1
+$EndComp
+$Comp
+L GND #PWR03
 U 1 1 4F684FA2
-P 4650 3250
-F 0 "#PWR01" H 4650 3250 30  0001 C CNN
-F 1 "GND" H 4650 3180 30  0001 C CNN
-	1    4650 3250
-	1    0    0    -1
-$EndComp
-$Comp
-L +3.3V #PWR02
+P 3150 3150
+F 0 "#PWR03" H 3150 3150 30  0001 C CNN
+F 1 "GND" H 3150 3080 30  0001 C CNN
+	1    3150 3150
+	1    0    0    -1
+$EndComp
+$Comp
+L +3.3V #PWR04
 U 1 1 4F684F91
-P 4650 2700
-F 0 "#PWR02" H 4650 2660 30  0001 C CNN
-F 1 "+3.3V" H 4650 2810 30  0000 C CNN
-	1    4650 2700
-	1    0    0    -1
-$EndComp
-$Comp
-L ATTINY85-P IC1
-U 1 1 4F684F67
-P 2000 2600
-F 0 "IC1" H 2100 2650 60  0000 C CNN
-F 1 "ATTINY85-P" H 4000 1850 60  0000 C CNN
-F 2 "DIP8" H 2100 1850 60  0001 C CNN
-	1    2000 2600
-	1    0    0    -1
-$EndComp
+P 3150 1050
+F 0 "#PWR04" H 3150 1010 30  0001 C CNN
+F 1 "+3.3V" H 3150 1160 30  0000 C CNN
+	1    3150 1050
+	1    0    0    -1
+$EndComp

Commit message: Working Code with a Three LED Eye
Uses software PWM and is still very much a work in progress. However it
is actually working and lovely and cylon like!
Parts:
- removed SW1: SW_PUSH, symbol SW_PUSH
- renumbered CON1 to CON?, IC1 to IC?
Connections:
- net GND: no longer CON?.6
Other:
- note removed: "PB2-5 are PWM Pins"
Changed lines of the file:
@@
-EESchema Schematic File Version 2  date 09/09/2013 14:06:59
+EESchema Schematic File Version 2  date 25/09/2013 14:24:36
 LIBS:power
 LIBS:device
@@
 LIBS:contrib
 LIBS:valves
-LIBS:Larson15cm_1-cache
 EELAYER 25  0
 EELAYER END
@@
 Sheet 1 1
 Title "noname.sch"
-Date "9 sep 2013"
+Date "25 sep 2013"
 Rev ""
 Comp ""
@@
 $EndDescr
 Wire Wire Line
-	4300 2750 4350 2750
-Wire Wire Line
-	4350 2750 4350 3250
-Wire Wire Line
-	4350 3250 2050 3250
-Wire Wire Line
-	6225 2325 6225 2050
-Wire Wire Line
-	6225 2050 5675 2050
+	1600 4800 1600 3000
+Wire Wire Line
+	1500 2900 1500 4700
+Wire Wire Line
+	1400 4600 1400 2800
+Wire Wire Line
+	1300 4500 1300 2700
+Wire Wire Line
+	4300 2750 4400 2750
+Wire Wire Line
+	4400 2750 4400 3250
 Wire Wire Line
 	4300 1850 4850 1850
@@
 Wire Wire Line
 	2050 2700 2050 3250
+Wire Wire Line
+	2050 3250 4400 3250
 Wire Wire Line
 	1900 2900 1500 2900
@@
 Wire Wire Line
 	1600 3900 4700 3900
-Wire Wire Line
-	1600 4800 1600 3000
-Wire Wire Line
-	1400 4600 1400 2800
 Connection ~ 5200 4800
 Connection ~ 5450 4500
-Wire Wire Line
-	1300 4500 1300 2700
 Connection ~ 6950 4000
 Wire Wire Line
@@
 Connection ~ 4700 4600
 Connection ~ 4950 4700
-Wire Wire Line
-	1500 2900 1500 4700
 Connection ~ 1500 3800
 Connection ~ 1300 3600
@@
 Wire Wire Line
 	2000 1075 2000 1350
-Wire Wire Line
-	4300 2450 5200 2450
-Wire Wire Line
-	5200 2450 5200 2700
-Wire Wire Line
-	5200 2700 5400 2700
-$Comp
-L GND #PWR01
-U 1 1 521BAF71
-P 6000 2700
-F 0 "#PWR01" H 6000 2700 30  0001 C CNN
-F 1 "GND" H 6000 2630 30  0001 C CNN
-	1    6000 2700
-	1    0    0    -1
-$EndComp
-$Comp
-L SW_PUSH SW1
-U 1 1 521BAF63
-P 5700 2700
-F 0 "SW1" H 5850 2810 50  0000 C CNN
-F 1 "SW_PUSH" H 5700 2620 50  0000 C CNN
-	1    5700 2700
-	1    0    0    -1
-$EndComp
-$Comp
-L GND #PWR02
-U 1 1 521BAC4F
-P 6225 2325
-F 0 "#PWR02" H 6225 2325 30  0001 C CNN
-F 1 "GND" H 6225 2255 30  0001 C CNN
-	1    6225 2325
-	1    0    0    -1
-$EndComp
-Text Notes 3075 2200 0    60   ~ 0
-PB2-5 are PWM Pins
-$Comp
-L AVR-ISP-6 CON1
+$Comp
+L AVR-ISP-6 CON?
 U 1 1 521BAA0B
 P 5550 1950
-F 0 "CON1" H 5470 2190 50  0000 C CNN
+F 0 "CON?" H 5470 2190 50  0000 C CNN
 F 1 "AVR-ISP-6" H 5310 1720 50  0000 L BNN
 F 2 "AVR-ISP-6" V 5030 1990 50  0001 C CNN
@@
 $EndComp
 $Comp
-L ATTINY2313-P IC1
+L ATTINY2313-P IC?
 U 1 1 521BA8AA
 P 3150 2150
-F 0 "IC1" H 2300 3100 60  0000 C CNN
+F 0 "IC?" H 2300 3100 60  0000 C CNN
 F 1 "ATTINY2313-P" H 3750 1300 60  0000 C CNN
 F 2 "DIP20" H 2350 1300 60  0001 C CNN
@@
 $EndComp
 $Comp
-L GND #PWR03
+L GND #PWR01
 U 1 1 4F684FA2
 P 3150 3150
-F 0 "#PWR03" H 3150 3150 30  0001 C CNN
+F 0 "#PWR01" H 3150 3150 30  0001 C CNN
 F 1 "GND" H 3150 3080 30  0001 C CNN
 	1    3150 3150
@@
 $EndComp
 $Comp
-L +3.3V #PWR04
+L +3.3V #PWR02
 U 1 1 4F684F91
 P 3150 1050
-F 0 "#PWR04" H 3150 1010 30  0001 C CNN
+F 0 "#PWR02" H 3150 1010 30  0001 C CNN
 F 1 "+3.3V" H 3150 1160 30  0000 C CNN
 	1    3150 1050
